File: 100W Amplifier IS/100W Amplifier IS.kicad_pcb (KiCad board)
At the start: 2 copper layers, 85.3 x 85.6 mm, 22 parts, among them J1 AudioJack2, J2 Back Pins (Odd), J3 Front Pins (Even), J4 -36DC Conn, J5 +36DC Conn, J6 Speaker Outupt, J7 -36 Switch Terminal, J8 +36 Switch Terminal

Commit message: gerber files
Parts:
- added ?: , , F.Cu at (115.6, 48.4)
- added ?: , , F.Cu at (175.4, 42.2)
- added ?: , , F.Cu at (115.5, 87.3)
- added REF**: MountingHole_2.2mm_M2_DIN965_Pad, MountingHole:MountingHole_2.2mm_M2_DIN965_Pad, F.Cu at (189.5, 115.7)
- added REF**: MountingHole_2.2mm_M2_DIN965_Pad, MountingHole:MountingHole_2.2mm_M2_DIN965_Pad, F.Cu at (175.4, 42.2)
- added REF**: MountingHole_2.2mm_M2_DIN965_Pad, MountingHole:MountingHole_2.2mm_M2_DIN965_Pad, F.Cu at (115.6, 48.4)
- added REF**: MountingHole_2.2mm_M2_DIN965_Pad, MountingHole:MountingHole_2.2mm_M2_DIN965_Pad, F.Cu at (115.5, 87.3)
- J1: value AudioJack2 -> Audio Jack
